Commit message: asd

File: gazebo_sim/franka_description_sim/robots/dual_panda_example.urdf.xacro (robot description, xacro)
@@ -3,6 +3,6 @@
   <xacro:arg name="arm_id_1" default="panda_1" />
   <xacro:arg name="arm_id_2" default="panda_2" />
-  <xacro:include filename="$(find franka_description)/robots/panda_arm.xacro"/>
-  <xacro:include filename="$(find franka_description)/robots/hand.xacro"/>
+  <xacro:include filename="$(find franka_description_sim)/robots/panda_arm.xacro"/>
+  <xacro:include filename="$(find franka_description_sim)/robots/hand.xacro"/>
   <!-- box shaped table as base for the 2 Pandas -->
   <link name="base">
@@ -30,6 +30,6 @@
   <xacro:hand ns="$(arg arm_id_2)" rpy="0 0 ${-pi/4}" connected_to="$(arg arm_id_2)_link8" safety_distance="0.03"/>
   <!-- Gazebo control -->
-  <xacro:include filename="$(find franka_description)/robots/panda.gazebo.xacro"/>
-  <xacro:include filename="$(find franka_description)/robots/panda.control.xacro"/>
+  <xacro:include filename="$(find franka_description_sim)/robots/panda.gazebo.xacro"/>
+  <xacro:include filename="$(find franka_description_sim)/robots/panda.control.xacro"/>
   <!-- Panda 1 gazebo -->
   <!--     arm     -->

File: gazebo_sim/franka_description_sim/robots/hand.urdf.xacro (robot description, xacro)
@@ -5,6 +5,6 @@
   <xacro:include filename="hand.xacro"/>
   <xacro:if value="$(arg use_gazebo_sim)">
-    <xacro:include filename="$(find franka_description)/robots/panda.gazebo.xacro"/>
-    <xacro:include filename="$(find franka_description)/robots/panda.control.xacro"/>
+    <xacro:include filename="$(find franka_description_sim)/robots/panda.gazebo.xacro"/>
+    <xacro:include filename="$(find franka_description_sim)/robots/panda.control.xacro"/>
   </xacro:if>
   <xacro:hand ns="panda" rpy="0 0 ${-pi/4}" connected_to="panda_link8" safety_distance="0.03"

File: gazebo_sim/franka_description_sim/robots/hand.xacro (robot description, xacro)
@@ -15,5 +15,5 @@
       <visual>
         <geometry>
-          <mesh filename="file://$(find franka_description)/meshes/visual/hand.dae"/>
+          <mesh filename="file://$(find franka_description_sim)/meshes/visual/hand.dae"/>
         </geometry>
       </visual>
@@ -59,5 +59,5 @@
         <collision>
           <geometry>
-            <mesh filename="file://$(find franka_description)/meshes/collision/hand.stl"/>
+            <mesh filename="file://$(find franka_description_sim)/meshes/collision/hand.stl"/>
           </geometry>
         </collision>
@@ -74,5 +74,5 @@
       <visual>
         <geometry>
-          <mesh filename="file://$(find franka_description)/meshes/visual/finger.dae"/>
+          <mesh filename="file://$(find franka_description_sim)/meshes/visual/finger.dae"/>
         </geometry>
       </visual>
@@ -80,5 +80,5 @@
         <collision>
           <geometry>
-            <mesh filename="file://$(find franka_description)/meshes/collision/finger.stl"/>
+            <mesh filename="file://$(find franka_description_sim)/meshes/collision/finger.stl"/>
           </geometry>
         </collision>
@@ -96,5 +96,5 @@
         <origin xyz="0 0 0" rpy="0 0 ${pi}"/>
         <geometry>
-          <mesh filename="file://$(find franka_description)/meshes/visual/finger.dae"/>
+          <mesh filename="file://$(find franka_description_sim)/meshes/visual/finger.dae"/>
         </geometry>
       </visual>
@@ -103,5 +103,5 @@
           <origin xyz="0 0 0" rpy="0 0 ${pi}"/>
           <geometry>
-            <mesh filename="file://$(find franka_description)/meshes/collision/finger.stl"/>
+            <mesh filename="file://$(find franka_description_sim)/meshes/collision/finger.stl"/>
           </geometry>
         </collision>

File: gazebo_sim/franka_description_sim/robots/panda_arm.urdf.xacro (robot description, xacro)
@@ -5,8 +5,8 @@
   <xacro:arg name="use_gazebo_sim" default="false"/>
   <xacro:arg name="parent" default="world"/>
-  <xacro:include filename="$(find franka_description)/robots/panda_arm.xacro" />
+  <xacro:include filename="$(find franka_description_sim)/robots/panda_arm.xacro" />
   <xacro:if value="$(arg use_gazebo_sim)">
-    <xacro:include filename="$(find franka_description)/robots/panda.gazebo.xacro"/>
-    <xacro:include filename="$(find franka_description)/robots/panda.control.xacro"/>
+    <xacro:include filename="$(find franka_description_sim)/robots/panda.gazebo.xacro"/>
+    <xacro:include filename="$(find franka_description_sim)/robots/panda.control.xacro"/>
   </xacro:if>
   <!-- <link name="world"/> -->

File: gazebo_sim/omtp_lecture1/urdf/omtp_custom_factory.urdf.xacro (robot description, xacro)
@@ -30,9 +30,9 @@
   <xacro:arg name="parent" default="robot1_pedestal_link"/>
   <!-- Load panda arm and hand -->
-  <xacro:include filename="$(find franka_description)/robots/panda_arm.xacro" />
-  <xacro:include filename="$(find franka_description)/robots/hand.xacro"/>
+  <xacro:include filename="$(find franka_description_sim)/robots/panda_arm.xacro" />
+  <xacro:include filename="$(find franka_description_sim)/robots/hand.xacro"/>
   <!-- Load gazebo control -->
-  <xacro:include filename="$(find franka_description)/robots/panda.gazebo.xacro"/>
-  <xacro:include filename="$(find franka_description)/robots/panda.control.xacro"/>
+  <xacro:include filename="$(find franka_description_sim)/robots/panda.gazebo.xacro"/>
+  <xacro:include filename="$(find franka_description_sim)/robots/panda.control.xacro"/>
   <!-- Panda 1 -->
   <xacro:panda_arm xyz="0.05 0 0.95" rpy="0 0 0" connected_to="$(arg parent)" arm_id="$(arg arm_id_1)" safety_distance="0.03" use_cylinder_collision_model="$(arg use_cylinder_collision_model)"/>
