Commit message: df

File: gazebo_sim/franka_description_sim/robots/panda_arm.xacro (robot description, xacro)
@@ -4,5 +4,5 @@
   <!-- safety_distance: Minimum safety distance in [m] by which the collision volumes are expanded and which is enforced during robot motions -->
   <!-- arm_id: Namespace of the panda arm. Serves to differentiate between arms in case of multiple instances. -->
-  <xacro:macro name="panda_arm" params="arm_id:='panda' description_pkg:='franka_description'
+  <xacro:macro name="panda_arm" params="arm_id:='panda' description_pkg:='franka_description_sim'
     connected_to:='' xyz:='0 0 0' rpy:='0 0 0' safety_distance:=0 use_cylinder_collision_model:='true'">
     <xacro:unless value="${not connected_to}">
