Commit message: sd

File: gazebo_sim/omtp_factory_moveit_config/config/omtp_factory.urdf.xacro (robot description, xacro)
@@ -7,8 +7,8 @@
     <!-- <xacro:include filename="$(find ariac_sensors)/models/basic_logical_camera/model.sdf" /> -->
     <!-- Import control_xacro -->
-    <!-- <xacro:include filename="omtp_factory.ros2_control.xacro" />
-    <xacro:omtp_factory_ros2_control name="FakeSystem" initial_positions_file="$(arg initial_positions_file)"/> -->
-    <xacro:include filename="omtp_factory.ros2_gazebo_control.xacro" />
-    <xacro:omtp_factory_ros2_gazebo_control name="GazeboSystem" initial_positions_file="$(arg initial_positions_file)"/>
+    <xacro:include filename="omtp_factory.ros2_control.xacro" />
+    <xacro:omtp_factory_ros2_control name="FakeSystem" initial_positions_file="$(arg initial_positions_file)"/>
+    <!-- <xacro:include filename="omtp_factory.ros2_gazebo_control.xacro" />
+    <xacro:omtp_factory_ros2_gazebo_control name="GazeboSystem" initial_positions_file="$(arg initial_positions_file)"/> -->
     <xacro:property name="M_PI"              value="3.1415926535897931"/>
 	<xacro:arg      name="camera_pose_trans" default="0 1.2 2.0"/>

File: gazebo_sim/omtp_lecture1/urdf/omtp_custom_factory.urdf.xacro (robot description, xacro)
@@ -9,12 +9,12 @@
   <!-- ==================================================== -->
   <!-- world -->
-  <link name="world"/>
+  <!-- <link name="world"/> -->
   <!-- world_interface. Makes it convenient to move the whole environment according to the world origin -->
   <link name="world_interface"/>
   <!-- world<->world_interface joint -->
-  <joint name="world_interface_to_world" type="fixed">
+  <!-- <joint name="world_interface_to_world" type="fixed">
     <parent link="world"/>
     <child link="world_interface"/>
-  </joint>
+  </joint> -->
   <!-- <xacro:include filename="$(find aau_lab_ros_models)/urdf/fib14/fib14.urdf.xacro"/>
   <xacro:fib14_urdf fib14_parent="world_interface"/> -->
@@ -28,5 +28,6 @@
   <xacro:arg name="use_cylinder_collision_model" default="true"/>
   <xacro:arg name="use_gazebo_sim" default="true"/>
-  <xacro:arg name="parent" default="robot1_pedestal_link"/>
+  <!-- <xacro:arg name="parent" default="robot1_pedestal_link"/> -->
+  <xacro:arg name="parent" default="world_interface"/>
   <!-- Load panda arm and hand -->
   <xacro:include filename="$(find franka_description_sim)/robots/panda_arm.xacro" />
@@ -36,13 +37,17 @@
   <xacro:include filename="$(find franka_description_sim)/robots/panda.control.xacro"/>
   <!-- Panda 1 -->
-  <xacro:panda_arm xyz="0.05 0 0.95" rpy="0 0 0" connected_to="$(arg parent)" arm_id="$(arg arm_id_1)" safety_distance="0.03" use_cylinder_collision_model="$(arg use_cylinder_collision_model)"/>
+  <xacro:panda_arm xyz="0.0 0 0.0" rpy="0 0 0" connected_to="$(arg parent)" arm_id="$(arg arm_id_1)" safety_distance="0.03" use_cylinder_collision_model="$(arg use_cylinder_collision_model)"/>
   <xacro:hand ns="$(arg arm_id_1)" rpy="0 0 ${-pi/4}" connected_to="$(arg arm_id_1)_link8" safety_distance="0.03" use_cylinder_collision_model="$(arg use_cylinder_collision_model)"/>
   <xacro:arm_gazebo arm_id="$(arg arm_id_1)"/>
   <xacro:arm_control arm_id="$(arg arm_id_1)"/>
-  <xacro:include filename="$(find external_ros_models)/urdf/robot_pedestal/robot_pedestal.urdf.xacro"/>
+  <!-- <xacro:panda_arm xyz="0.05 0 0.95" rpy="0 0 0" connected_to="$(arg parent)" arm_id="$(arg arm_id_1)" safety_distance="0.03" use_cylinder_collision_model="$(arg use_cylinder_collision_model)"/>
+  <xacro:hand ns="$(arg arm_id_1)" rpy="0 0 ${-pi/4}" connected_to="$(arg arm_id_1)_link8" safety_distance="0.03" use_cylinder_collision_model="$(arg use_cylinder_collision_model)"/>
+  <xacro:arm_gazebo arm_id="$(arg arm_id_1)"/>
+  <xacro:arm_control arm_id="$(arg arm_id_1)"/> -->
+  <!-- <xacro:include filename="$(find external_ros_models)/urdf/robot_pedestal/robot_pedestal.urdf.xacro"/>
   <xacro:robot_pedestal_urdf pedestal_prefix="robot1_" pedestal_parent="world_interface" pedestal_height="0.95">
-    <origin xyz="-0.6 1.5 0.0" rpy="0 0 0"/>
-  </xacro:robot_pedestal_urdf>
-  <xacro:include filename="$(find aau_lab_ros_models)/urdf/festo_straight_module/festo_straight_module.urdf.xacro"/>
+    <origin xyz="0.0 0.0 0.0" rpy="0 0 0"/>
+  </xacro:robot_pedestal_urdf> -->
+  <!-- <xacro:include filename="$(find aau_lab_ros_models)/urdf/festo_straight_module/festo_straight_module.urdf.xacro"/>
 	<xacro:festo_module_urdf module_prefix="module1_" festo_module_parent="world_interface">
 		<origin xyz="0.0 1.5 0.0" rpy="0 0 0.0"/>
@@ -54,5 +59,5 @@
 			<origin xyz="0.0 1.5 1.0" rpy="0 0 0" />
 		</xacro:conveyor>
-	</xacro:if>
+	</xacro:if> -->
   <!-- franka robot 2 -->
   <!-- <xacro:arg name="arm_id_2" default="panda2"/>

Commit message: corrected namespace of camera

File: gazebo_sim/omtp_factory_moveit_config/config/omtp_factory.urdf.xacro (robot description, xacro)
@@ -7,13 +7,13 @@
     <!-- <xacro:include filename="$(find ariac_sensors)/models/basic_logical_camera/model.sdf" /> -->
     <!-- Import control_xacro -->
-    <xacro:include filename="omtp_factory.ros2_control.xacro" />
-    <xacro:omtp_factory_ros2_control name="FakeSystem" initial_positions_file="$(arg initial_positions_file)"/>
-    <!-- <xacro:include filename="omtp_factory.ros2_gazebo_control.xacro" />
-    <xacro:omtp_factory_ros2_gazebo_control name="GazeboSystem" initial_positions_file="$(arg initial_positions_file)"/> -->
+    <!-- <xacro:include filename="omtp_factory.ros2_control.xacro" />
+    <xacro:omtp_factory_ros2_control name="FakeSystem" initial_positions_file="$(arg initial_positions_file)"/> -->
+    <xacro:include filename="omtp_factory.ros2_gazebo_control.xacro" />
+    <xacro:omtp_factory_ros2_gazebo_control name="GazeboSystem" initial_positions_file="$(arg initial_positions_file)"/>
     <xacro:property name="M_PI"              value="3.1415926535897931"/>
 	<xacro:arg      name="camera_pose_trans" default="0 1.2 2.0"/>
 	<xacro:arg      name="camera_pose_rot"   default="0.0 ${M_PI/2.0} 0.0"/>
     <xacro:include filename="$(find omtp_lecture5)/urdf/camera/_d435.urdf.xacro" />
-		<xacro:sensor_d435 name="camera" topics_ns="camera" parent="world_interface" publish_pointcloud="true">
+		<xacro:sensor_d435 name="camera" topics_ns="camera/" parent="world_interface" publish_pointcloud="true">
 			<origin xyz="$(arg camera_pose_trans)" rpy="$(arg camera_pose_rot)" />
 		</xacro:sensor_d435>

File: gazebo_sim/omtp_lecture1/urdf/omtp_custom_factory.urdf.xacro (robot description, xacro)
@@ -28,6 +28,6 @@
   <xacro:arg name="use_cylinder_collision_model" default="true"/>
   <xacro:arg name="use_gazebo_sim" default="true"/>
-  <!-- <xacro:arg name="parent" default="robot1_pedestal_link"/> -->
-  <xacro:arg name="parent" default="world_interface"/>
+  <xacro:arg name="parent" default="robot1_pedestal_link"/>
+  <!-- <xacro:arg name="parent" default="world_interface"/> -->
   <!-- Load panda arm and hand -->
   <xacro:include filename="$(find franka_description_sim)/robots/panda_arm.xacro" />
@@ -37,17 +37,17 @@
   <xacro:include filename="$(find franka_description_sim)/robots/panda.control.xacro"/>
   <!-- Panda 1 -->
-  <xacro:panda_arm xyz="0.0 0 0.0" rpy="0 0 0" connected_to="$(arg parent)" arm_id="$(arg arm_id_1)" safety_distance="0.03" use_cylinder_collision_model="$(arg use_cylinder_collision_model)"/>
+  <!-- <xacro:panda_arm xyz="0.0 0 0.0" rpy="0 0 0" connected_to="$(arg parent)" arm_id="$(arg arm_id_1)" safety_distance="0.03" use_cylinder_collision_model="$(arg use_cylinder_collision_model)"/>
+  <xacro:hand ns="$(arg arm_id_1)" rpy="0 0 ${-pi/4}" connected_to="$(arg arm_id_1)_link8" safety_distance="0.03" use_cylinder_collision_model="$(arg use_cylinder_collision_model)"/>
+  <xacro:arm_gazebo arm_id="$(arg arm_id_1)"/>
+  <xacro:arm_control arm_id="$(arg arm_id_1)"/> -->
+  <xacro:panda_arm xyz="0.05 0.0 0.95" rpy="0 0 0" connected_to="$(arg parent)" arm_id="$(arg arm_id_1)" safety_distance="0.03" use_cylinder_collision_model="$(arg use_cylinder_collision_model)"/>
   <xacro:hand ns="$(arg arm_id_1)" rpy="0 0 ${-pi/4}" connected_to="$(arg arm_id_1)_link8" safety_distance="0.03" use_cylinder_collision_model="$(arg use_cylinder_collision_model)"/>
   <xacro:arm_gazebo arm_id="$(arg arm_id_1)"/>
   <xacro:arm_control arm_id="$(arg arm_id_1)"/>
-  <!-- <xacro:panda_arm xyz="0.05 0 0.95" rpy="0 0 0" connected_to="$(arg parent)" arm_id="$(arg arm_id_1)" safety_distance="0.03" use_cylinder_collision_model="$(arg use_cylinder_collision_model)"/>
-  <xacro:hand ns="$(arg arm_id_1)" rpy="0 0 ${-pi/4}" connected_to="$(arg arm_id_1)_link8" safety_distance="0.03" use_cylinder_collision_model="$(arg use_cylinder_collision_model)"/>
-  <xacro:arm_gazebo arm_id="$(arg arm_id_1)"/>
-  <xacro:arm_control arm_id="$(arg arm_id_1)"/> -->
-  <!-- <xacro:include filename="$(find external_ros_models)/urdf/robot_pedestal/robot_pedestal.urdf.xacro"/>
+  <xacro:include filename="$(find external_ros_models)/urdf/robot_pedestal/robot_pedestal.urdf.xacro"/>
   <xacro:robot_pedestal_urdf pedestal_prefix="robot1_" pedestal_parent="world_interface" pedestal_height="0.95">
-    <origin xyz="0.0 0.0 0.0" rpy="0 0 0"/>
-  </xacro:robot_pedestal_urdf> -->
-  <!-- <xacro:include filename="$(find aau_lab_ros_models)/urdf/festo_straight_module/festo_straight_module.urdf.xacro"/>
+    <origin xyz="-0.6 1.5 0.0" rpy="0 0 0"/>
+  </xacro:robot_pedestal_urdf>
+  <xacro:include filename="$(find aau_lab_ros_models)/urdf/festo_straight_module/festo_straight_module.urdf.xacro"/>
 	<xacro:festo_module_urdf module_prefix="module1_" festo_module_parent="world_interface">
 		<origin xyz="0.0 1.5 0.0" rpy="0 0 0.0"/>
@@ -59,5 +59,5 @@
 			<origin xyz="0.0 1.5 1.0" rpy="0 0 0" />
 		</xacro:conveyor>
-	</xacro:if> -->
+	</xacro:if>
   <!-- franka robot 2 -->
   <!-- <xacro:arg name="arm_id_2" default="panda2"/>

File: gazebo_sim/omtp_lecture5/urdf/camera/_d435.urdf.xacro (robot description, xacro)
@@ -9,5 +9,5 @@
   <!--File includes-->
   <xacro:include filename="$(find omtp_lecture5)/urdf/camera/rgbd.gazebo.xacro"/>
-  <xacro:macro name="sensor_d435" params="name:=camera topics_ns:=camera parent *origin publish_pointcloud:=true">
+  <xacro:macro name="sensor_d435" params="name:=camera topics_ns:=camera/ parent *origin publish_pointcloud:=true">
     <xacro:property name="M_PI" value="3.1415926535897931" />
     <!-- The following values are approximate, and the camera node

File: gazebo_sim/omtp_lecture5/urdf/camera/rgbd.gazebo.xacro (robot description, xacro)
@@ -184,12 +184,12 @@
       <colorUpdateRate>30.0</colorUpdateRate>
       <infraredUpdateRate>1.0</infraredUpdateRate>
-      <depthTopicName>aligned_depth_to_color/image_raw</depthTopicName>
-      <depthCameraInfoTopicName>depth/camera_info</depthCameraInfoTopicName>
-      <colorTopicName>color/image_raw</colorTopicName>
-      <colorCameraInfoTopicName>color/camera_info</colorCameraInfoTopicName>
-      <infrared1TopicName>infra1/image_raw</infrared1TopicName>
-      <infrared1CameraInfoTopicName>infra1/camera_info</infrared1CameraInfoTopicName>
-      <infrared2TopicName>infra2/image_raw</infrared2TopicName>
-      <infrared2CameraInfoTopicName>infra2/camera_info</infrared2CameraInfoTopicName>
+      <depthTopicName>camera/aligned_depth_to_color/image_raw</depthTopicName>
+      <depthCameraInfoTopicName>camera/depth/camera_info</depthCameraInfoTopicName>
+      <colorTopicName>camera/color/image_raw</colorTopicName>
+      <colorCameraInfoTopicName>camera/color/camera_info</colorCameraInfoTopicName>
+      <infrared1TopicName>camera/infra1/image_raw</infrared1TopicName>
+      <infrared1CameraInfoTopicName>camera/infra1/camera_info</infrared1CameraInfoTopicName>
+      <infrared2TopicName>camera/infra2/image_raw</infrared2TopicName>
+      <infrared2CameraInfoTopicName>camera/infra2/camera_info</infrared2CameraInfoTopicName>
       <colorOpticalframeName>camera_color_optical_frame</colorOpticalframeName>
       <depthOpticalframeName>${depth_optical_frame}</depthOpticalframeName>
@@ -199,5 +199,5 @@
       <rangeMaxDepth>3.0</rangeMaxDepth>
       <pointCloud>true</pointCloud>
-      <pointCloudTopicName>depth/color/points</pointCloudTopicName>
+      <pointCloudTopicName>camera/depth/color/points</pointCloudTopicName>
       <pointCloudCutoff>0.3</pointCloudCutoff>
       </plugin>
