Commit message: as

File: gazebo_sim/omtp_factory_moveit_config/config/omtp_factory.ros2_control.xacro (robot description, xacro)
@@ -8,90 +8,90 @@
                 <plugin>mock_components/GenericSystem</plugin>
             </hardware>
-            <joint name="panda1_joint1">
+            <joint name="panda_joint1">
                 <command_interface name="position"/>
                 <command_interface name="velocity"/>
                 <command_interface name="effort"/>
                 <state_interface name="position">
-                  <param name="initial_value">${initial_positions['panda1_joint1']}</param>
+                  <param name="initial_value">${initial_positions['panda_joint1']}</param>
                 </state_interface>
                 <state_interface name="velocity"/>
                 <state_interface name="acceleration"/>
             </joint>
-            <joint name="panda1_joint2">
+            <joint name="panda_joint2">
                 <command_interface name="position"/>
                 <command_interface name="velocity"/>
                 <command_interface name="effort"/>
                 <state_interface name="position">
-                  <param name="initial_value">${initial_positions['panda1_joint2']}</param>
+                  <param name="initial_value">${initial_positions['panda_joint2']}</param>
                 </state_interface>
                 <state_interface name="velocity"/>
                 <state_interface name="acceleration"/>
             </joint>
-            <joint name="panda1_joint3">
+            <joint name="panda_joint3">
                 <command_interface name="position"/>
                 <command_interface name="velocity"/>
                 <command_interface name="effort"/>
                 <state_interface name="position">
-                  <param name="initial_value">${initial_positions['panda1_joint3']}</param>
+                  <param name="initial_value">${initial_positions['panda_joint3']}</param>
                 </state_interface>
                 <state_interface name="velocity"/>
                 <state_interface name="acceleration"/>
             </joint>
-            <joint name="panda1_joint4">
+            <joint name="panda_joint4">
                 <command_interface name="position"/>
                 <command_interface name="velocity"/>
                 <command_interface name="effort"/>
                 <state_interface name="position">
-                  <param name="initial_value">${initial_positions['panda1_joint4']}</param>
+                  <param name="initial_value">${initial_positions['panda_joint4']}</param>
                 </state_interface>
                 <state_interface name="velocity"/>
                 <state_interface name="acceleration"/>
             </joint>
-            <joint name="panda1_joint5">
+            <joint name="panda_joint5">
                 <command_interface name="position"/>
                 <command_interface name="velocity"/>
                 <command_interface name="effort"/>
                 <state_interface name="position">
-                  <param name="initial_value">${initial_positions['panda1_joint5']}</param>
+                  <param name="initial_value">${initial_positions['panda_joint5']}</param>
                 </state_interface>
                 <state_interface name="velocity"/>
                 <state_interface name="acceleration"/>
             </joint>
-            <joint name="panda1_joint6">
+            <joint name="panda_joint6">
                 <command_interface name="position"/>
                 <command_interface name="velocity"/>
                 <command_interface name="effort"/>
                 <state_interface name="position">
-                  <param name="initial_value">${initial_positions['panda1_joint6']}</param>
+                  <param name="initial_value">${initial_positions['panda_joint6']}</param>
                 </state_interface>
                 <state_interface name="velocity"/>
                 <state_interface name="acceleration"/>
             </joint>
-            <joint name="panda1_joint7">
+            <joint name="panda_joint7">
                 <command_interface name="position"/>
                 <command_interface name="velocity"/>
                 <command_interface name="effort"/>
                 <state_interface name="position">
-                  <param name="initial_value">${initial_positions['panda1_joint7']}</param>
+                  <param name="initial_value">${initial_positions['panda_joint7']}</param>
                 </state_interface>
                 <state_interface name="velocity"/>
                 <state_interface name="acceleration"/>
             </joint>
-            <joint name="panda1_finger_joint1">
+            <joint name="panda_finger_joint1">
                 <command_interface name="position"/>
                 <command_interface name="velocity"/>
                 <command_interface name="effort"/>
                 <state_interface name="position">
-                  <param name="initial_value">${initial_positions['panda1_finger_joint1']}</param>
+                  <param name="initial_value">${initial_positions['panda_finger_joint1']}</param>
                 </state_interface>
                 <state_interface name="velocity"/>
                 <state_interface name="acceleration"/>
             </joint>
-            <joint name="panda1_finger_joint2">
+            <joint name="panda_finger_joint2">
                 <command_interface name="position"/>
                 <command_interface name="velocity"/>
                 <command_interface name="effort"/>
                 <state_interface name="position">
-                  <param name="initial_value">${initial_positions['panda1_finger_joint2']}</param>
+                  <param name="initial_value">${initial_positions['panda_finger_joint2']}</param>
                 </state_interface>
                 <state_interface name="velocity"/>
