Commit message: asd

File: gazebo_sim/omtp_factory_moveit_config/config/omtp_factory.ros2_gazebo_control.xacro (robot description, xacro)
@@ -7,68 +7,68 @@
       <plugin>gazebo_ros2_control/GazeboSystem</plugin>
     </hardware>
-    <joint name="panda1_joint1">
+    <joint name="panda_joint1">
       <command_interface name="effort" />
       <state_interface name="velocity" />
       <state_interface name="position">
-                  <param name="initial_value">${initial_positions['panda1_finger_joint1']}</param>
+                  <param name="initial_value">${initial_positions['panda_finger_joint1']}</param>
                 </state_interface>
     </joint>
-    <joint name="panda1_joint2">
+    <joint name="panda_joint2">
       <command_interface name="effort" />
       <state_interface name="velocity" />
       <state_interface name="position">
-                  <param name="initial_value">${initial_positions['panda1_finger_joint1']}</param>
+                  <param name="initial_value">${initial_positions['panda_finger_joint1']}</param>
                 </state_interface>
     </joint>
-    <joint name="panda1_joint3">
+    <joint name="panda_joint3">
       <command_interface name="effort" />
       <state_interface name="velocity" />
       <state_interface name="position">
-                  <param name="initial_value">${initial_positions['panda1_finger_joint1']}</param>
+                  <param name="initial_value">${initial_positions['panda_finger_joint1']}</param>
                 </state_interface>
     </joint>
-    <joint name="panda1_joint4">
+    <joint name="panda_joint4">
       <command_interface name="effort" />
       <state_interface name="velocity" />
       <state_interface name="position">
-                  <param name="initial_value">${initial_positions['panda1_finger_joint1']}</param>
+                  <param name="initial_value">${initial_positions['panda_finger_joint1']}</param>
                 </state_interface>
     </joint>
-    <joint name="panda1_joint5">
+    <joint name="panda_joint5">
       <command_interface name="effort" />
       <state_interface name="velocity" />
       <state_interface name="position">
-                  <param name="initial_value">${initial_positions['panda1_finger_joint1']}</param>
+                  <param name="initial_value">${initial_positions['panda_finger_joint1']}</param>
                 </state_interface>
     </joint>
-    <joint name="panda1_joint6">
+    <joint name="panda_joint6">
       <command_interface name="effort" />
       <state_interface name="velocity" />
       <state_interface name="position">
-                  <param name="initial_value">${initial_positions['panda1_finger_joint1']}</param>
+                  <param name="initial_value">${initial_positions['panda_finger_joint1']}</param>
                 </state_interface>
     </joint>
-    <joint name="panda1_joint7">
+    <joint name="panda_joint7">
       <command_interface name="effort" />
       <state_interface name="velocity" />
       <state_interface name="position">
-                  <param name="initial_value">${initial_positions['panda1_finger_joint1']}</param>
+                  <param name="initial_value">${initial_positions['panda_finger_joint1']}</param>
                 </state_interface>
     </joint>
-    <joint name="panda1_finger_joint1">
+    <joint name="panda_finger_joint1">
                 <command_interface name="position"/>
                 <command_interface name="velocity"/>
                 <command_interface name="effort"/>
                 <state_interface name="position">
-                  <param name="initial_value">${initial_positions['panda1_finger_joint1']}</param>
+                  <param name="initial_value">${initial_positions['panda_finger_joint1']}</param>
                 </state_interface>
                 <state_interface name="velocity"/>
             </joint>
-            <joint name="panda1_finger_joint2">
+            <joint name="panda_finger_joint2">
                 <command_interface name="position"/>
                 <command_interface name="velocity"/>
                 <command_interface name="effort"/>
                 <state_interface name="position">
-                  <param name="initial_value">${initial_positions['panda1_finger_joint2']}</param>
+                  <param name="initial_value">${initial_positions['panda_finger_joint2']}</param>
                 </state_interface>
                 <state_interface name="velocity"/>

File: gazebo_sim/omtp_factory_moveit_config/config/omtp_factory.urdf.xacro (robot description, xacro)
@@ -7,8 +7,8 @@
     <!-- <xacro:include filename="$(find ariac_sensors)/models/basic_logical_camera/model.sdf" /> -->
     <!-- Import control_xacro -->
-    <!-- <xacro:include filename="omtp_factory.ros2_control.xacro" />
-    <xacro:omtp_factory_ros2_control name="FakeSystem" initial_positions_file="$(arg initial_positions_file)"/> -->
-    <xacro:include filename="omtp_factory.ros2_gazebo_control.xacro" />
-    <xacro:omtp_factory_ros2_gazebo_control name="GazeboSystem" initial_positions_file="$(arg initial_positions_file)"/>
+    <xacro:include filename="omtp_factory.ros2_control.xacro" />
+    <xacro:omtp_factory_ros2_control name="FakeSystem" initial_positions_file="$(arg initial_positions_file)"/>
+    <!-- <xacro:include filename="omtp_factory.ros2_gazebo_control.xacro" />
+    <xacro:omtp_factory_ros2_gazebo_control name="GazeboSystem" initial_positions_file="$(arg initial_positions_file)"/> -->
     <xacro:property name="M_PI"              value="3.1415926535897931"/>
 	<xacro:arg      name="camera_pose_trans" default="0 1.2 2.0"/>

File: gazebo_sim/omtp_lecture1/urdf/omtp_custom_factory.urdf.xacro (robot description, xacro)
@@ -25,5 +25,5 @@
   <xacro:panda_arm arm_id="$(arg arm_id_1)" connected_to="${robot1_pedestal_link}"  xyz="${0 -0.5 1}" safety_distance="0.03"/>
   <xacro:hand ns="$(arg arm_id_1)" rpy="0 0 ${-pi/4}" connected_to="$(arg arm_id_1)_link8" safety_distance="0.03"/> -->
-  <xacro:arg name="arm_id_1" default="panda1"/>
+  <xacro:arg name="arm_id_1" default="panda"/>
   <xacro:arg name="use_cylinder_collision_model" default="true"/>
   <xacro:arg name="use_gazebo_sim" default="true"/>

Commit message: indenting

File: gazebo_sim/omtp_factory_moveit_config/config/omtp_factory.ros2_gazebo_control.xacro (robot description, xacro)
@@ -4,57 +4,57 @@
         <xacro:property name="initial_positions" value="${load_yaml(initial_positions_file)['initial_positions']}"/>
         <ros2_control name="GazeboSystem" type="system">
-    <hardware>
-      <plugin>gazebo_ros2_control/GazeboSystem</plugin>
-    </hardware>
-    <joint name="panda_joint1">
-      <command_interface name="effort" />
-      <state_interface name="velocity" />
-      <state_interface name="position">
-                  <param name="initial_value">${initial_positions['panda_finger_joint1']}</param>
-                </state_interface>
-    </joint>
-    <joint name="panda_joint2">
-      <command_interface name="effort" />
-      <state_interface name="velocity" />
-      <state_interface name="position">
-                  <param name="initial_value">${initial_positions['panda_finger_joint1']}</param>
-                </state_interface>
-    </joint>
-    <joint name="panda_joint3">
-      <command_interface name="effort" />
-      <state_interface name="velocity" />
-      <state_interface name="position">
-                  <param name="initial_value">${initial_positions['panda_finger_joint1']}</param>
-                </state_interface>
-    </joint>
-    <joint name="panda_joint4">
-      <command_interface name="effort" />
-      <state_interface name="velocity" />
-      <state_interface name="position">
-                  <param name="initial_value">${initial_positions['panda_finger_joint1']}</param>
-                </state_interface>
-    </joint>
-    <joint name="panda_joint5">
-      <command_interface name="effort" />
-      <state_interface name="velocity" />
-      <state_interface name="position">
-                  <param name="initial_value">${initial_positions['panda_finger_joint1']}</param>
-                </state_interface>
-    </joint>
-    <joint name="panda_joint6">
-      <command_interface name="effort" />
-      <state_interface name="velocity" />
-      <state_interface name="position">
-                  <param name="initial_value">${initial_positions['panda_finger_joint1']}</param>
-                </state_interface>
-    </joint>
-    <joint name="panda_joint7">
-      <command_interface name="effort" />
-      <state_interface name="velocity" />
-      <state_interface name="position">
-                  <param name="initial_value">${initial_positions['panda_finger_joint1']}</param>
-                </state_interface>
-    </joint>
-    <joint name="panda_finger_joint1">
+            <hardware>
+              <plugin>gazebo_ros2_control/GazeboSystem</plugin>
+            </hardware>
+            <joint name="panda_joint1">
+              <command_interface name="effort" />
+              <state_interface name="velocity" />
+              <state_interface name="position">
+                          <param name="initial_value">${initial_positions['panda_finger_joint1']}</param>
+                        </state_interface>
+            </joint>
+            <joint name="panda_joint2">
+              <command_interface name="effort" />
+              <state_interface name="velocity" />
+              <state_interface name="position">
+                          <param name="initial_value">${initial_positions['panda_finger_joint1']}</param>
+                        </state_interface>
+            </joint>
+            <joint name="panda_joint3">
+              <command_interface name="effort" />
+              <state_interface name="velocity" />
+              <state_interface name="position">
+                          <param name="initial_value">${initial_positions['panda_finger_joint1']}</param>
+                        </state_interface>
+            </joint>
+            <joint name="panda_joint4">
+              <command_interface name="effort" />
+              <state_interface name="velocity" />
+              <state_interface name="position">
+                          <param name="initial_value">${initial_positions['panda_finger_joint1']}</param>
+                        </state_interface>
+            </joint>
+            <joint name="panda_joint5">
+              <command_interface name="effort" />
+              <state_interface name="velocity" />
+              <state_interface name="position">
+                          <param name="initial_value">${initial_positions['panda_finger_joint1']}</param>
+                        </state_interface>
+            </joint>
+            <joint name="panda_joint6">
+              <command_interface name="effort" />
+              <state_interface name="velocity" />
+              <state_interface name="position">
+                          <param name="initial_value">${initial_positions['panda_finger_joint1']}</param>
+                        </state_interface>
+            </joint>
+            <joint name="panda_joint7">
+              <command_interface name="effort" />
+              <state_interface name="velocity" />
+              <state_interface name="position">
+                          <param name="initial_value">${initial_positions['panda_finger_joint1']}</param>
+                        </state_interface>
+            </joint>
+            <joint name="panda_finger_joint1">
                 <command_interface name="position"/>
                 <command_interface name="velocity"/>
@@ -74,10 +74,10 @@
                 <state_interface name="velocity"/>
             </joint>
-  </ros2_control>
-  <gazebo>
-    <plugin filename="libgazebo_ros2_control.so" name="gazebo_ros2_control">
-      <parameters>$(find omtp_factory_moveit_config)/config/ros2_controllers_gazebo.yaml</parameters>
-    </plugin>
-  </gazebo>
+        </ros2_control>
+        <gazebo>
+          <plugin filename="libgazebo_ros2_control.so" name="gazebo_ros2_control">
+            <parameters>$(find omtp_factory_moveit_config)/config/ros2_controllers_gazebo.yaml</parameters>
+          </plugin>
+        </gazebo>
     </xacro:macro>
 </robot>
