Commit message: added static aruco cube to default urdf

File: gazebo_sim/gazebo_tests/models/aruco_cube/aruco_cube.gazebo.xacro (robot description, xacro)
@@ -1,24 +1,6 @@
 <?xml version="1.0"?>
-<robot xmlns:xacro="http://www.ros.org/wiki/xacro">
-  <xacro:macro name="aruco_cube_gazebo" params="prefix">
-    <gazebo reference="${prefix}drop_point">
-      <sensor name="${prefix}contact_sensor" type="contact">
-        <update_rate>10</update_rate>
-        <contact>
-          <collision>${prefix}base_link_collision</collision>
-        </contact>
-      </sensor>
-    </gazebo>
+<robot name="aruco_cube_gazebo" xmlns:xacro="http://www.ros.org/wiki/xacro">
     <gazebo>
       <static>true</static>
-<!--
-       <plugin name="${prefix}object_disposal_plugin" filename="libObjectDisposalPlugin.so">
-        <contact_sensor_name>${prefix}contact_sensor</contact_sensor_name>
-        <contact_side_normal>0 0 1</contact_side_normal>
-        <disposal_pose>0 0 0 0 0 0</disposal_pose>
-        <update_rate>1</update_rate>
-      </plugin>
- -->
      </gazebo>
-  </xacro:macro>
 </robot>

File: gazebo_sim/gazebo_tests/models/aruco_cube/aruco_cube.urdf.xacro (robot description, xacro)
@@ -1,23 +1,24 @@
 <?xml version="1.0"?>
-<robot name="aruco_cube">
-  <xacro:macro name="aruco_cube_macro" params="prefix">
-    <link name="link">
-      <inertial>
-        <origin xyz="0 0 0" rpy="0 0 0"/>
-        <mass value="0.25"/>
-        <inertia ixx="0.00001066664" ixy="0.0" ixz="0.0" iyy="0.00001066664" iyz="0.0" izz="0.00001066664"/>
-      </inertial>
-      <collision name="collision">
-        <origin xyz="0 0 0" rpy="0 0 0"/>
-        <geometry>
-          <mesh filename="model://aruco_cube/meshes/aruco_cube_8cm.dae"/>
-        </geometry>
-      </collision>
-      <visual name="visual">
-        <origin xyz="0 0 0" rpy="0 0 0"/>
-        <geometry>
-          <mesh filename="model://aruco_cube/meshes/aruco_cube_8cm.dae"/>
-        </geometry>
-      </visual>
+<robot name="aruco_cube" xmlns:xacro="http://www.ros.org/wiki/xacro">
+<xacro:macro name="aruco_cube_macro" params="*origin">
+  <link name="cube_link">
+    <inertial>
+      <origin xyz="0 0 0" rpy="0 0 0"/>
+      <mass value="0.25"/>
+      <inertia ixx="0.00001066664" ixy="0.0" ixz="0.0" iyy="0.00001066664" iyz="0.0" izz="0.00001066664"/>
+    </inertial>
+    <collision name="collision">
+      <origin xyz="0 0 0" rpy="0 0 0"/>
+      <geometry>
+        <mesh filename="model://aruco_cube/meshes/aruco_cube_8cm.dae"/>
+      </geometry>
+    </collision>
+    <visual name="visual">
+      <origin xyz="0 0 0" rpy="0 0 0"/>
+      <geometry>
+        <mesh filename="model://aruco_cube/meshes/aruco_cube_8cm.dae"/>
+      </geometry>
+    </visual>
+    <gazebo reference="cube_link">
       <velocity_decay>
         <linear value="0.0"/>
@@ -27,5 +28,11 @@
       <kinematic>0</kinematic>
       <gravity>1</gravity>
-    </link>
-  </xacro:macro>
+    </gazebo>
+  </link>
+  <joint name="aruco_cube_joint" type="fixed">
+    <xacro:insert_block name="origin" />
+    <parent link="world_interface"/>
+    <child link="cube_link"/>
+  </joint>
+</xacro:macro>
 </robot>

File: gazebo_sim/gazebo_tests/models/aruco_cube/aruco_cube.xacro (robot description, xacro)
@@ -1,10 +1,17 @@
 <?xml version="1.0"?>
 <robot name="aruco_cube" xmlns:xacro="http://www.ros.org/wiki/xacro">
-  <xacro:arg name="prefix" default="1_"/>
-  <!-- URDF -->
-  <xacro:include filename="$(find gazebo_tests)/models/aruco_cube/aruco_cube.urdf.xacro"/>
-  <xacro:aruco_cube_macro prefix="$(arg prefix)"/>
-  <!-- Gazebo -->
-  <!-- <xacro:include filename="$(find gazebo_tests)/models/aruco_cube/aruco_cube.gazebo.xacro"/>
-  <xacro:aruco_cube_gazebo prefix="$(arg prefix)"/> -->
+  <!-- <xacro:macro name="aruco_cube"> -->
+    <!-- <xacro:arg name="sufix" default="_1"/> -->
+    <!-- URDF -->
+    <xacro:include filename="$(find gazebo_tests)/models/aruco_cube/aruco_cube.urdf.xacro"/>
+    <xacro:aruco_cube_macro>
+      <origin xyz="0.0 0.0 0.0" rpy="0.0 0.0 0.0"/>
+    </xacro:aruco_cube_macro>
+    <xacro:robot_pedestal_urdf pedestal_prefix="$(arg pedestal_prefix)" pedestal_parent="$(arg pedestal_parent)" pedestal_height="$(arg pedestal_height)">
+    <origin xyz="0.5 1.8 0.0" rpy="0.0 0.0 0.0"/>
+  </xacro:robot_pedestal_urdf>
+    <!-- Gazebo -->
+    <xacro:include filename="$(find gazebo_tests)/models/aruco_cube/aruco_cube.gazebo.xacro"/>
+    <!-- <xacro:aruco_cube_gazebo /> -->
+  <!-- </xacro:macro> -->
 </robot>

File: gazebo_sim/omtp_lecture1/urdf/omtp_custom_factory.urdf.xacro (robot description, xacro)
@@ -41,4 +41,8 @@
   <xacro:arm_gazebo arm_id="$(arg arm_id_1)"/>
   <xacro:arm_control arm_id="$(arg arm_id_1)"/> -->
+  <xacro:include filename="$(find gazebo_tests)/models/aruco_cube/aruco_cube.urdf.xacro"/>
+  <xacro:aruco_cube_macro>
+      <origin xyz="0.0 1.2 1.2" rpy="0.0 0.0 0.0"/>
+  </xacro:aruco_cube_macro>
   <xacro:panda_arm xyz="0.05 0.0 0.95" rpy="0 0 0" connected_to="$(arg parent)" arm_id="$(arg arm_id_1)" safety_distance="0.03" use_cylinder_collision_model="$(arg use_cylinder_collision_model)"/>
   <xacro:hand ns="$(arg arm_id_1)" rpy="0 0 ${-pi/4}" connected_to="$(arg arm_id_1)_link8" safety_distance="0.03" use_cylinder_collision_model="$(arg use_cylinder_collision_model)"/>
