Commit message: made to xacro macro

File: gazebo_sim/gazebo_tests/models/aruco_cube/aruco_cube.urdf.xacro (robot description, xacro)
@@ -1,29 +1,31 @@
 <?xml version="1.0"?>
 <robot name="aruco_cube">
-  <link name="link">
-    <inertial>
-      <origin xyz="0 0 0" rpy="0 0 0"/>
-      <mass value="0.25"/>
-      <inertia ixx="0.00001066664" ixy="0.0" ixz="0.0" iyy="0.00001066664" iyz="0.0" izz="0.00001066664"/>
-    </inertial>
-    <collision name="collision">
-      <origin xyz="0 0 0" rpy="0 0 0"/>
-      <geometry>
-        <mesh filename="model://aruco_cube/meshes/aruco_cube_8cm.dae"/>
-      </geometry>
-    </collision>
-    <visual name="visual">
-      <origin xyz="0 0 0" rpy="0 0 0"/>
-      <geometry>
-        <mesh filename="model://aruco_cube/meshes/aruco_cube_8cm.dae"/>
-      </geometry>
-    </visual>
-    <velocity_decay>
-      <linear value="0.0"/>
-      <angular value="0.0"/>
-    </velocity_decay>
-    <self_collide>0</self_collide>
-    <kinematic>0</kinematic>
-    <gravity>1</gravity>
-  </link>
+  <xacro:macro name="aruco_cube_macro" params="prefix">
+    <link name="link">
+      <inertial>
+        <origin xyz="0 0 0" rpy="0 0 0"/>
+        <mass value="0.25"/>
+        <inertia ixx="0.00001066664" ixy="0.0" ixz="0.0" iyy="0.00001066664" iyz="0.0" izz="0.00001066664"/>
+      </inertial>
+      <collision name="collision">
+        <origin xyz="0 0 0" rpy="0 0 0"/>
+        <geometry>
+          <mesh filename="model://aruco_cube/meshes/aruco_cube_8cm.dae"/>
+        </geometry>
+      </collision>
+      <visual name="visual">
+        <origin xyz="0 0 0" rpy="0 0 0"/>
+        <geometry>
+          <mesh filename="model://aruco_cube/meshes/aruco_cube_8cm.dae"/>
+        </geometry>
+      </visual>
+      <velocity_decay>
+        <linear value="0.0"/>
+        <angular value="0.0"/>
+      </velocity_decay>
+      <self_collide>0</self_collide>
+      <kinematic>0</kinematic>
+      <gravity>1</gravity>
+    </link>
+  </xacro:macro>
 </robot>

File: gazebo_sim/gazebo_tests/models/aruco_cube/aruco_cube.xacro (robot description, xacro)
@@ -4,7 +4,7 @@
   <!-- URDF -->
   <xacro:include filename="$(find gazebo_tests)/models/aruco_cube/aruco_cube.urdf.xacro"/>
-  <xacro:bin_urdf prefix="$(arg prefix)"/>
+  <xacro:aruco_cube_macro prefix="$(arg prefix)"/>
   <!-- Gazebo -->
-  <xacro:include filename="$(find gazebo_tests)/models/aruco_cube/aruco_cube.gazebo.xacro"/>
-  <xacro:aruco_cube_gazebo prefix="$(arg prefix)"/>
+  <!-- <xacro:include filename="$(find gazebo_tests)/models/aruco_cube/aruco_cube.gazebo.xacro"/>
+  <xacro:aruco_cube_gazebo prefix="$(arg prefix)"/> -->
 </robot>

Commit message: fixed mesh naming

File: gazebo_sim/gazebo_tests/models/aruco_cube/aruco_cube.urdf.xacro (robot description, xacro)
@@ -11,5 +11,6 @@
       <origin xyz="0 0 0" rpy="0 0 0"/>
       <geometry>
-        <mesh filename="model://aruco_cube/meshes/aruco_cube_8cm.dae"/>
+        <!-- <mesh filename="file://aruco_cube/meshes/aruco_cube_8cm.dae"/> -->
+        <mesh filename="file://$(find gazebo_tests)/models/aruco_cube/meshes/aruco_cube_8cm.dae"/>
       </geometry>
     </collision>
@@ -17,5 +18,6 @@
       <origin xyz="0 0 0" rpy="0 0 0"/>
       <geometry>
-        <mesh filename="model://aruco_cube/meshes/aruco_cube_8cm.dae"/>
+        <!-- <mesh filename="file://aruco_cube/meshes/aruco_cube_8cm.dae"/> -->
+        <mesh filename="file://$(find gazebo_tests)/models/aruco_cube/meshes/aruco_cube_8cm.dae"/>
       </geometry>
     </visual>

File: gazebo_sim/omtp_lecture5/urdf/camera/_d435.urdf.xacro (robot description, xacro)
@@ -49,5 +49,4 @@
           <!-- <box size="${d435_cam_width} ${d435_cam_height} ${d435_cam_depth}"/> -->
           <mesh filename="file://$(find realsense2_description)/meshes/d435.dae" />
-          <!--<mesh filename="file://$(find realsense2_description)/meshes/d435/d435.dae" />-->
         </geometry>
         <material name="${name}_aluminum"/>
