Commit message: better

File: gazebo_sim/omtp_lecture5/urdf/camera/_d435.urdf.xacro (robot description, xacro)
@@ -33,5 +33,6 @@
     <!-- camera body, with origin at bottom screw mount -->
     <joint name="${name}_joint" type="fixed">
-      <origin xyz="0 1.2 2.0" rpy="0.0 ${M_PI/2.0} 0.0"/>
+      <!-- <origin xyz="0 0.0 0.0" rpy="0.0 0.0 0.0"/> -->
+      <xacro:insert_block name="origin"/>
       <parent link="${parent}"/>
       <child link="${name}_bottom_screw_frame" />
