Commit message: added offset for aruco code to tube grab pose, using tf link

File: manipulator/urdf/test_tube_w_holder/robot.urdf (robot description, URDF)
Before this commit: robot onshape, 2 links, 3 joints
Links:
- removed link aruco
- removed link grab
- added link single_test_tube_holder, mass 0; collision mesh filename=file:///home/intelnuc/sdl_ws/src/self_driving_lab/manipulat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; collision mesh filename=file:///home/intelnuc/sdl_ws/src/self_driving_lab/manipulat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
Joints:
- removed joint idk
- removed joint test
- joint single_test_tube_holder_joint: child aruco -> single_test_tube_holder
